File: kicad/VictronMP-II-FanController.kicad_sch (KiCad schematic)
At the start: 28 parts, among them J1 MultiPlus 1 FAN, J2 MultiPlus 2 FAN, J3 MultiPlus 3 FAN, J4 Noctua Fan 1, J5 Noctua Fan 2, J6 Noctua Fan 3, Q1 BC547B, Q2 BC547B, Q3 BC547B, U1 PC817, U2 PC817, U3 PC817, U4 Seeed XIAO ESP32-C6

Commit message: Adjusted resistors in schematic
Parts:
- removed R10, R8: 10k, Resistor_THT:R_Axial_DIN0207_L6.3mm_D2.5mm_P10.16mm_Horizontal, symbol FanCtrl:R
- R1, R2, R3: value 4.7k 0.5W -> 4.7k
Connections:
- net at R11.1, R7.1, R9.1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: now also R12.2
- net at Q3.2 (B), R11.2: no longer R12.2
Other:
- moved on the sheet: R12
